Commit message: Add web-based TonyPi digital twin, replace tonypi_sim
New digital_twin/ package: URDF-based simulator with a three.js browser
viewer, replacing the Open3D/PyBullet visualizer (laptop_mvp/tonypi_sim.py).

- Servo pulse <-> joint calibration derived from scripts/poses.json
  (stand-pose zero, 240 deg / 1000 pulses), clamped to robot_api limits
- Base URDF moved from laptop_mvp and extended with hip/ankle roll joints
- Floor-contact solver so leaning poses show a tilted torso, not floating feet
- Two channels: command (estimator/poses/sliders) and actual (read-only
  servo/status readback from robot_api), shown solid with the other as a ghost
- Stdlib HTTP + SSE server, CORS open; embeddable twin.js module, iframe
  mode, and optional FastAPI mount_twin()
- mediapose_est.py / yolo_est.py drive the twin with the exact servo pulses
  they send the robot (--twin-port, --no-browser, --twin-robot-url)
- Tests: tests/test_digital_twin.py; retarget/pipeline/mediapose tests
  moved to the new API

Co-Authored-By: Claude Sonnet 5.5 <noreply@anthropic.com>
Claude-Session: https://claude.ai/code/session_0126w7aHwV3VTJrp9Q2812Bd

File: digital_twin/tonypi.urdf (robot description, URDF)
Before this commit: robot tonypi, 16 links, 15 joints
Links:
- added link l_ankle_link, mass 0.04; visual box size=0.034 0.034 0.034
- added link l_hip_link, mass 0.04; visual box size=0.034 0.034 0.034
- added link r_ankle_link, mass 0.04; visual box size=0.034 0.034 0.034
- added link r_hip_link, mass 0.04; visual box size=0.034 0.034 0.034
Joints:
- removed joint l_ankle
- removed joint r_ankle
- added joint l_ankle_pitch: type revolute, parent l_shin, child l_ankle_link, origin xyz=0 0 -0.075 rpy=0 0 0, axis 0 1 0, limit lower=-2.0 upper=2.0 effort=4.0 velocity=4.0
- added joint l_ankle_roll: type revolute, parent l_ankle_link, child l_foot, origin xyz=0 0 0 rpy=0 0 0, axis 1 0 0, limit lower=-1.0 upper=1.0 effort=4.0 velocity=4.0
- added joint l_hip_roll: type revolute, parent pelvis, child l_hip_link, origin xyz=0 0.045 -0.028 rpy=0 0 0, axis 1 0 0, limit lower=-1.0 upper=1.0 effort=4.0 velocity=4.0
- added joint r_ankle_pitch: type revolute, parent r_shin, child r_ankle_link, origin xyz=0 0 -0.075 rpy=0 0 0, axis 0 1 0, limit lower=-2.0 upper=2.0 effort=4.0 velocity=4.0
- added joint r_ankle_roll: type revolute, parent r_ankle_link, child r_foot, origin xyz=0 0 0 rpy=0 0 0, axis 1 0 0, limit lower=-1.0 upper=1.0 effort=4.0 velocity=4.0
- added joint r_hip_roll: type revolute, parent pelvis, child r_hip_link, origin xyz=0 -0.045 -0.028 rpy=0 0 0, axis 1 0 0, limit lower=-1.0 upper=1.0 effort=4.0 velocity=4.0
- joint l_hip_pitch: limit lower=-1.57 upper=1.57 effort=4.0 velocity=4.0 -> lower=-2.1 upper=2.1 effort=4.0 velocity=4.0; origin xyz=0 0.045 -0.028 rpy=0 0 0 -> xyz=0 0 0 rpy=0 0 0; parent pelvis -> l_hip_link
- joint l_knee: limit lower=-1.57 upper=1.57 effort=4.0 velocity=4.0 -> lower=-2.1 upper=2.1 effort=4.0 velocity=4.0
- joint r_hip_pitch: limit lower=-1.57 upper=1.57 effort=4.0 velocity=4.0 -> lower=-2.1 upper=2.1 effort=4.0 velocity=4.0; origin xyz=0 -0.045 -0.028 rpy=0 0 0 -> xyz=0 0 0 rpy=0 0 0; parent pelvis -> r_hip_link
- joint r_knee: limit lower=-1.57 upper=1.57 effort=4.0 velocity=4.0 -> lower=-2.1 upper=2.1 effort=4.0 velocity=4.0
