Commit message: streaming for robot api

File: digital_twin/tonypi.urdf (robot description, URDF)
Before this commit: robot tonypi, 20 links, 19 joints
Links:
- link l_forearm: geometry collision box size=0.024 0.028 0.080; visual box size=0.022 0.004 0.012
- link r_forearm: geometry collision box size=0.024 0.028 0.080; visual box size=0.022 0.004 0.012
Joints:
- joint l_elbow: axis 0 1 0 -> 1 0 0
- joint r_elbow: axis 0 1 0 -> -1 0 0

Commit message: Fix digital twin elbow axes and model depth conflicts
Model servos 6 and 14 as mirrored inward-sweeping hinges, align estimator kinematics and command limits, and remove coplanar model surfaces and floor/ghost depth conflicts.

Fixes #19

File: digital_twin/tonypi.urdf (robot description, URDF)
Before this commit: robot tonypi, 20 links, 19 joints
Links:
- link l_ankle_link: geometry visual box size=0.032 0.032 0.034
- link l_hip_link: geometry visual box size=0.032 0.032 0.034
- link l_shin: geometry collision box size=0.034 0.034 0.075; visual box size=0.034 0.034 0.070
- link l_upper_arm: geometry collision box size=0.028 0.032 0.080; visual box size=0.028 0.032 0.076
- link r_ankle_link: geometry visual box size=0.032 0.032 0.034
- link r_hip_link: geometry visual box size=0.032 0.032 0.034
- link r_shin: geometry collision box size=0.034 0.034 0.075; visual box size=0.034 0.034 0.070
- link r_upper_arm: geometry collision box size=0.028 0.032 0.080; visual box size=0.028 0.032 0.076
Joints:
- joint l_elbow: axis 0 1 0 -> 1 0 0
- joint r_elbow: axis 0 1 0 -> -1 0 0
